Commit message: add trace movement

File: urdfs/drone_x.urdf (robot description, URDF)
Before this commit: robot drone, 9 links, 8 joints
Joints:
- joint l1: origin xyz=0.5 0.0 0.0 -> xyz=0.35 0.35 0.0
- joint l2: origin xyz=0.0 0.5 0.0 -> xyz=-0.35 0.35 0.0
- joint l3: origin xyz=-0.5 0.0 0.0 -> xyz=0.35 -0.35 0.0
- joint l4: origin xyz=0.0 -0.5 0.0 -> xyz=-0.35 -0.35 0.0
